File: wada_pcb_60.kicad_pcb (KiCad board)
At the start: 2 copper layers, 284.7 x 94.2 mm, 243 parts, among them J1 USB_C_Receptacle_USB2.0_16P, J2 USB_A, J3 USB_A, U1 XC6206PxxxMR, U2 STM32F072C8T6, U3 MIC2026-2BN, U4 FE1.1, U5 SRV05-4, U6 SRV05-4, U7 SRV05-4, U8 74AHCT1G125, Y1 12MHz

Commit message: wired up the LEDS, rows, and columns!
Parts:
- moved JP1 2.94 mm to (146.0, 171.7), turned to -90 degrees
- moved C13 0.73 mm to (83.6, 144.8)
- moved C22 0.40 mm to (91.8, 145.3)
- moved C46 0.32 mm to (127.8, 169.9)
- moved LED16 0.32 mm to (129.9, 171.4)
- moved R14 0.20 mm to (144.9, 181.3)
Connections:
- C23 pad 1: /PORT1_PWR -> /PORT2_PWR
- C24 pad 1: /PORT1_PWR -> /PORT2_PWR
- C25 pad 1: /PORT1_PWR -> /PORT2_PWR
- C26 pad 1: /PORT2_PWR -> /PORT1_PWR
- C27 pad 1: /PORT2_PWR -> /PORT1_PWR
- C28 pad 1: /PORT2_PWR -> /PORT1_PWR
- J2 pad 1: /PORT1_PWR -> /PORT2_PWR
- J2 pad 2: D_USB1- -> D_USB2-
- J2 pad 3: D_USB1+ -> D_USB2+
- J3 pad 1: /PORT2_PWR -> /PORT1_PWR
- J3 pad 2: D_USB2- -> D_USB1-
- J3 pad 3: D_USB2+ -> D_USB1+
- U6 pad 3: D_USB1+ -> D_USB2+
- U6 pad 4: D_USB1- -> D_USB2-
- U6 pad 5: /PORT1_PWR -> /PORT2_PWR
- U7 pad 3: D_USB2+ -> D_USB1+
- U7 pad 4: D_USB2- -> D_USB1-
- U7 pad 5: /PORT2_PWR -> /PORT1_PWR
Routing:
- net VCC: track 138.4 -> 799.7 mm, vias 6 -> 15
- net ROW2: track 0.00 -> 319.0 mm, vias 0 -> 6
- net ROW1: track 0.00 -> 289.2 mm, vias 0 -> 6
- net ROW0: track 0.00 -> 265.2 mm, vias 0 -> 6
- net ROW4: track 0.00 -> 261.7 mm, vias 0 -> 2
- net ROW3: track 0.00 -> 257.9 mm
- net COL1: track 5.17 -> 118.6 mm, vias 0 -> 1
- net COL2: track 7.14 -> 97.3 mm, vias 0 -> 1
- net COL9: track 4.76 -> 93.8 mm
- net COL4: track 24.1 -> 111.5 mm
- net COL0: track 10.2 -> 97.0 mm, vias 0 -> 2
- net COL8: track 9.74 -> 96.3 mm, vias 2 -> 0
- net COL6: track 0.00 -> 85.7 mm
- net COL11: track 0.00 -> 84.1 mm
- net COL12: track 11.9 -> 96.0 mm
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
Commit message: done! missing the reset switch!
Parts:
- moved JP1 20.7 mm to (137.5, 190.5), turned to 0 degrees
- moved C46 2.21 mm to (125.6, 170.1)
- moved LED16 2.10 mm to (127.8, 171.3)
- moved R14 1.10 mm to (144.9, 182.4)
Connections:
- U2 pad 13: /A3 -> ROW0
- U2 pad 14: /A4 -> ROW1
- U2 pad 15: /A5 -> ROW2
- U2 pad 16: /A6 -> ROW3
- U2 pad 21: /B10 -> ROW4
- U2 pad 25: /B12 -> COL2
- U2 pad 26: /B13 -> COL0
- U2 pad 27: /B14 -> COL1
- U2 pad 28: /B15 -> COL13
- U2 pad 29: /A8 -> COL12
- U2 pad 30: /A9 -> COL11
- U2 pad 31: /A10 -> COL3
- U2 pad 37: /A14 -> COL10
- U2 pad 38: /A15 -> COL9
- U2 pad 39: /B3 -> COL8
- U2 pad 40: /B4 -> COL7
- U2 pad 41: /B5 -> COL6
- U2 pad 42: /B6 -> COL5
- U2 pad 43: /B7 -> COL4
Routing:
- net COL13: track 100.0 -> 320.1 mm
- net COL12: track 96.0 -> 295.8 mm
- net COL11: track 84.1 -> 265.7 mm
- net ROW0: track 265.2 -> 440.0 mm, vias 6 -> 8
- net COL10: track 65.0 -> 221.7 mm
- net ROW1: track 289.2 -> 442.2 mm, vias 6 -> 8
- net COL9: track 93.8 -> 230.7 mm
- net ROW2: track 319.0 -> 441.9 mm, vias 6 -> 8
- net ROW3: track 257.9 -> 375.8 mm, vias 0 -> 6
- net COL8: track 96.3 -> 213.5 mm
- net COL7: track 65.0 -> 162.8 mm
- net COL6: track 85.7 -> 163.9 mm
- net COL0: track 97.0 -> 172.6 mm, vias 2 -> 3
- net COL5: track 61.2 -> 120.2 mm
- net COL1: track 118.6 -> 166.6 mm, vias 1 -> 2
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
Commit message: review time!
Parts:
- removed JP1: BOOT0, Connector_PinHeader_2.54mm:PinHeader_1x02_P2.54mm_Vertical
- removed R5: 10kR, Resistor_SMD:R_0603_1608Metric
- added BOOT_SW1: SW_SPST, Button_Switch_SMD:SW_SPST_TL3342, B.Cu at (159.1, 171.2)
- added C47: 100nF, Capacitor_SMD:C_0603_1608Metric, B.Cu at (135.4, 188.2)
- added RESET_SW1: SW_SPST, Button_Switch_SMD:SW_SPST_TL3342, B.Cu at (149.3, 188.7)
- moved R14 11.3 mm to (151.4, 173.1), turned to 180 degrees
- moved LED16 2.90 mm to (124.9, 171.3)
- moved C46 2.90 mm to (122.7, 170.1)
- moved J3 0.80 mm to (166.0, 104.9)
- moved J2 0.78 mm to (127.9, 104.9)
- moved U6 0.78 mm to (127.9, 116.8)
- moved U7 0.40 mm to (166.0, 116.7)
Routing:
- net GND: track 121.2 -> 145.3 mm, vias 57 -> 60
- net STM32_3V3: track 107.3 -> 125.6 mm, vias 5 -> 7
- net NRST: track 3.54 -> 21.6 mm
- net BOOT0: track 17.4 -> 29.5 mm
- net GNDPWR: track 367.8 -> 374.3 mm
- net VCC: track 801.8 -> 804.7 mm
- net Net-(LED15-DOUT): track 25.1 -> 22.2 mm
- net D_USB2+: track 98.4 -> 96.8 mm
- net D_USB2-: track 97.0 -> 95.4 mm
- net D_USB1-: track 132.6 -> 131.8 mm
- net D_USB1+: track 134.1 -> 133.3 mm
- net /PORT1_PWR: track 68.6 -> 68.0 mm
