File: wada_pcb_60.kicad_pcb (KiCad board)
At the start: 2 copper layers, 284.7 x 94.2 mm, 244 parts, among them J1 USB_C_Receptacle_USB2.0_16P, J2 USB_A, J3 USB_A, U1 XC6206PxxxMR, U2 STM32F072C8T6, U3 MIC2026-2BN, U4 FE1.1, U5 SRV05-4, U6 SRV05-4, U7 SRV05-4, U8 74AHCT1G125, Y1 12MHz

Commit message: Changed USB type-A and LED parts
Parts:
- removed C46: 100nF, Capacitor_SMD:C_0603_1608Metric
- J2, J3: footprint cipulot_parts:USB-SMT-04F-S1-B1-R9A -> JING_USB-A:JING 903-231A2031S10100
- LED1, LED10, LED11, LED12, LED13, LED14, LED15, LED16, LED2, LED3, LED4, LED5, LED6, LED7, LED8, LED9: value WS2812_2020 -> SK6812MINI; footprint PCM_marbastlib-various:LED_WS2812_2020 -> LED_SMD:LED_SK6812MINI_PLCC4_3.5x3.5mm_P1.75mm
- moved C37 6.00 mm to (293.8, 116.7), turned to 0 degrees
- moved C40 5.86 mm to (180.7, 116.7), turned to 0 degrees
- moved C39 5.85 mm to (223.5, 116.8), turned to 0 degrees
- moved C38 5.67 mm to (256.2, 116.7), turned to 0 degrees
- moved C42 5.52 mm to (106.4, 117.1), turned to 0 degrees
- moved C43 5.50 mm to (67.5, 117.1), turned to 0 degrees
- moved C31 5.24 mm to (174.7, 169.5)
- moved C36 5.13 mm to (325.0, 117.8)
- moved C33 5.11 mm to (250.3, 169.6)
- moved C35 5.10 mm to (322.5, 169.6)
- moved C34 5.05 mm to (287.5, 169.6)
- moved C44 5.02 mm to (65.4, 169.5)
- moved C45 5.02 mm to (99.9, 169.5)
- moved C32 4.84 mm to (218.6, 169.6)
- moved J2 4.22 mm to (127.9, 109.1), turned to 0 degrees
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Routing:
- net GND: track 145.3 -> 108.2 mm, vias 60 -> 67
- net VCC: track 804.7 -> 786.9 mm
- net Net-(LED14-DOUT): track 38.1 -> 33.4 mm
- net Net-(LED11-DOUT): track 37.3 -> 33.4 mm
- net ROW0: track 440.0 -> 436.3 mm
- net Net-(LED15-DOUT): track 22.2 -> 18.9 mm
- net COL13: track 320.1 -> 317.5 mm
- net Net-(D7-A): track 3.68 -> 6.27 mm
- net STM32_3V3: track 125.6 -> 123.0 mm
- net Net-(LED2-DOUT): track 31.4 -> 28.9 mm
- net COL0: track 172.6 -> 170.8 mm
- net Net-(D58-A): track 11.8 -> 9.96 mm
- net D_USB2-: track 95.4 -> 93.8 mm
- net COL2: track 132.3 -> 130.8 mm
- net Net-(LED8-DOUT): track 31.4 -> 29.9 mm
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
Commit message: checking phase
Parts:
- added C46: 100nF, Capacitor_SMD:C_0603_1608Metric, B.Cu at (118.6, 170.0)
- added G***: LOGO, cipulot_parts:Penguin_logo, B.Cu at (269.9, 128.9)
- added G***: LOGO, cipulot_parts:qmk_logo, B.Cu at (289.7, 188.2)
- added REF**: KB_LOGO, Keyboard_Logo:KB_LOGO, F.Cu at (166.0, 183.3)
- added REF**: KB_LOGO, Keyboard_Logo:KB_LOGO, F.Cu at (213.5, 183.3)
- added REF**: KB_LOGO, Keyboard_Logo:KB_LOGO, F.Cu at (189.7, 183.2)
- LED1, LED10, LED11, LED12, LED13, LED14, LED15, LED16, LED2, LED3, LED4, LED5, LED6, LED7, LED8, LED9: footprint LED_SMD:LED_SK6812MINI_PLCC4_3.5x3.5mm_P1.75mm -> LED_SK6812MINI_HS:LED_SK6812MINI_HAND_SOLDER_3.5x3.5mm_P1.75mm
- moved LED10 4.34 mm to (180.3, 114.8), turned to 90 degrees
- moved C40 3.30 mm to (184.0, 116.6)
- moved C44 2.90 mm to (68.3, 169.4)
- moved LED14 2.17 mm to (68.4, 173.2), turned to -90 degrees
- moved LED6 1.43 mm to (324.9, 114.0), turned to 90 degrees
- moved LED3 1.28 mm to (250.3, 173.3), turned to -90 degrees
- moved LED15 1.22 mm to (100.0, 173.3), turned to -90 degrees
- moved LED4 1.22 mm to (287.6, 173.3), turned to -90 degrees
- moved LED5 1.21 mm to (322.6, 173.3), turned to -90 degrees
- moved C31 1.15 mm to (175.8, 169.4)
- moved LED7 1.05 mm to (289.5, 114.9), turned to 90 degrees
- moved LED12 1.04 mm to (102.5, 115.3), turned to 90 degrees
- moved LED8 1.04 mm to (252.3, 115.0), turned to 90 degrees
- moved LED9 1.02 mm to (219.5, 115.0), turned to 90 degrees
- moved LED2 0.96 mm to (219.1, 173.3), turned to -90 degrees
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Routing:
- net GND: track 108.2 -> 146.1 mm, vias 67 -> 77
- net Net-(LED10-DOUT): track 39.4 -> 45.7 mm
- net VCC: track 786.9 -> 792.4 mm
- net Net-(LED13-DOUT): track 68.0 -> 72.4 mm
- net Net-(LED6-DOUT): track 33.1 -> 36.3 mm
- net Net-(LED1-DOUT): track 41.2 -> 44.3 mm
- net Net-(LED12-DOUT): track 36.3 -> 39.4 mm
- net Net-(LED15-DOUT): track 18.9 -> 21.5 mm
- net Net-(LED8-DOUT): track 29.9 -> 32.5 mm
- net Net-(LED3-DOUT): track 34.5 -> 37.0 mm
- net Net-(LED4-DOUT): track 32.2 -> 34.6 mm
- net Net-(LED7-DOUT): track 34.5 -> 36.9 mm
- net Net-(LED2-DOUT): track 28.9 -> 30.7 mm
- net Net-(LED11-DOUT): track 33.4 -> 34.7 mm
- net Net-(LED10-DIN): track 40.2 -> 39.0 mm
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Other:
- board text added: "A gift to:"
- board text added: "OK/Fail?"
- board text added: "Revision:"
